File: Wiring Schematic/Wiring Schematic/Wiring Schematic.kicad_sch (KiCad schematic)
At the start: 11 parts

Commit message: edition
Connections:
- net at M?.1 (PWM): no longer A?.21 (D6)
- net at U?.10 (IN3): now also A?.22 (D7); no longer A?.24 (D9)
- net at U?.11 (EnB): now also A?.21 (D6); no longer A?.25 (D10)
- net at U?.6 (EnA): now also A?.24 (D9); no longer A?.26 (D11)
Changed lines of the file:
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@@
 (kicad_sch (version 20211123) (generator eeschema)
   (paper "A4")
-  (wire (pts (xy 99.06 120.65) (xy 101.6 120.65))
-    (stroke (width 0) (type default) (color 0 0 0 0))
+  (junction (at 99.06 123.19) (diameter 0) (color 0 0 0 0)
   )
-  (wire (pts (xy 99.06 110.49) (xy 128.27 110.49))
+  (wire (pts (xy 106.68 105.41) (xy 106.68 107.95))
     (stroke (width 0) (type default) (color 0 0 0 0))
   )
@@
     (stroke (width 0) (type default) (color 0 0 0 0))
   )
-  (wire (pts (xy 106.68 85.09) (xy 106.68 105.41))
+  (wire (pts (xy 99.06 118.11) (xy 115.57 118.11))
     (stroke (width 0) (type default) (color 0 0 0 0))
   )
@@
     (stroke (width 0) (type default) (color 0 0 0 0))
   )
-  (wire (pts (xy 106.68 105.41) (xy 128.27 105.41))
+  (wire (pts (xy 115.57 118.11) (xy 115.57 113.03))
     (stroke (width 0) (type default) (color 0 0 0 0))
   )
@@
     (stroke (width 0) (type default) (color 0 0 0 0))
   )
-  (wire (pts (xy 104.14 121.92) (xy 104.14 123.19))
+  (wire (pts (xy 99.06 123.19) (xy 114.3 123.19))
     (stroke (width 0) (type default) (color 0 0 0 0))
   )
-  (wire (pts (xy 99.06 118.11) (xy 128.27 118.11))
+  (wire (pts (xy 111.76 107.95) (xy 111.76 113.03))
     (stroke (width 0) (type default) (color 0 0 0 0))
   )
-  (wire (pts (xy 101.6 121.92) (xy 104.14 121.92))
+  (wire (pts (xy 99.06 110.49) (xy 128.27 110.49))
     (stroke (width 0) (type default) (color 0 0 0 0))
   )
-  (wire (pts (xy 102.87 123.19) (xy 102.87 120.65))
+  (wire (pts (xy 128.27 105.41) (xy 106.68 105.41))
+    (stroke (width 0) (type default) (color 0 0 0 0))
+  )
+  (wire (pts (xy 99.06 113.03) (xy 111.76 113.03))
+    (stroke (width 0) (type default) (color 0 0 0 0))
+  )
+  (wire (pts (xy 118.11 123.19) (xy 128.27 123.19))
+    (stroke (width 0) (type default) (color 0 0 0 0))
+  )
+  (wire (pts (xy 115.57 113.03) (xy 128.27 113.03))
     (stroke (width 0) (type default) (color 0 0 0 0))
   )
@@
     (stroke (width 0) (type default) (color 0 0 0 0))
   )
-  (wire (pts (xy 101.6 120.65) (xy 101.6 121.92))
+  (wire (pts (xy 118.11 120.65) (xy 118.11 123.19))
     (stroke (width 0) (type default) (color 0 0 0 0))
   )
@@
     (stroke (width 0) (type default) (color 0 0 0 0))
   )
-  (wire (pts (xy 99.06 107.95) (xy 104.14 107.95))
+  (wire (pts (xy 99.06 120.65) (xy 118.11 120.65))
     (stroke (width 0) (type default) (color 0 0 0 0))
   )
-  (wire (pts (xy 104.14 107.95) (xy 104.14 115.57))
+  (wire (pts (xy 99.06 107.95) (xy 106.68 107.95))
     (stroke (width 0) (type default) (color 0 0 0 0))
   )
-  (wire (pts (xy 99.06 113.03) (xy 128.27 113.03))
+  (wire (pts (xy 114.3 121.92) (xy 114.3 123.19))
     (stroke (width 0) (type default) (color 0 0 0 0))
   )
@@
     (stroke (width 0) (type default) (color 0 0 0 0))
   )
-  (wire (pts (xy 104.14 115.57) (xy 128.27 115.57))
+  (wire (pts (xy 97.79 123.19) (xy 99.06 123.19))
     (stroke (width 0) (type default) (color 0 0 0 0))
   )
-  (wire (pts (xy 104.14 123.19) (xy 128.27 123.19))
+  (wire (pts (xy 114.3 121.92) (xy 121.92 121.92))
     (stroke (width 0) (type default) (color 0 0 0 0))
   )
-  (wire (pts (xy 99.06 123.19) (xy 102.87 123.19))
+  (wire (pts (xy 128.27 107.95) (xy 111.76 107.95))
+    (stroke (width 0) (type default) (color 0 0 0 0))
+  )
+  (wire (pts (xy 121.92 120.65) (xy 128.27 120.65))
     (stroke (width 0) (type default) (color 0 0 0 0))
   )
@@
     (stroke (width 0) (type default) (color 0 0 0 0))
   )
-  (wire (pts (xy 102.87 120.65) (xy 128.27 120.65))
+  (wire (pts (xy 121.92 121.92) (xy 121.92 120.65))
     (stroke (width 0) (type default) (color 0 0 0 0))
   )
